Commit message: refactor():更改gripper关节名，由joint*更改为gripper_joint*

File: piper_moveit/piper_moveit/piper_with_gripper_moveit/config/piper.ros2_control.xacro (robot description, xacro)
@@ -50,8 +50,8 @@
                 <state_interface name="velocity"/>
             </joint>
-            <joint name="joint8">
+            <joint name="gripper_joint2">
                 <command_interface name="position"/>
                 <state_interface name="position">
-                  <param name="initial_value">${initial_positions['joint8']}</param>
+                  <param name="initial_value">${initial_positions['gripper_joint2']}</param>
                 </state_interface>
                 <state_interface name="velocity"/>

File: piper_moveit/piper_x_moveit/piper_x_with_gripper_moveit/config/piper_x_description.ros2_control.xacro (robot description, xacro)
@@ -50,8 +50,8 @@
                 <state_interface name="velocity"/>
             </joint>
-            <joint name="joint8">
+            <joint name="gripper_joint2">
                 <command_interface name="position"/>
                 <state_interface name="position">
-                  <param name="initial_value">${initial_positions['joint8']}</param>
+                  <param name="initial_value">${initial_positions['gripper_joint2']}</param>
                 </state_interface>
                 <state_interface name="velocity"/>
